File: src_files/hdmi_mipi_2.sch (KiCad schematic (older format))
At the start: 37 parts, among them J1 HDMI-019S, J7 XF2M60151AH, U9 TC358870XBG_NOK_, Y3 CRYSTAL_48MHZ

Commit message: updated all files and production files as well
Parts:
- FB4: footprint Barrel - Audio Connectors:BEADC2012X105N -> Inductor_SMD:L_0603_1608Metric
Changed lines of the file:
@@
 F 0 "FB4" V 7728 1050 39  0000 C CNN
 F 1 "Ferrite_Bead_Small" V 7779 1050 50  0001 C CNN
-F 2 "Barrel - Audio Connectors:BEADC2012X105N" V 7855 1050 50  0001 C CNN
+F 2 "Inductor_SMD:L_0603_1608Metric" V 7855 1050 50  0001 C CNN
 F 3 "~" H 7925 1050 50  0001 C CNN
 F 4 "BLM21PG220SN1" V 7796 1050 30  0000 C CNN "MPN"
