File: src_files/hdmi_to_mipi-dsi_converter.sch (KiCad schematic (older format))
At the start: 42 parts, among them J2 HDMI-019S, J5 XF2M60151AH, U4 TC358870XBG_NOK_, Y1 CRYSTAL_48MHZ

Commit message: updated all files and production files as well
Parts:
- FB1: footprint Barrel - Audio Connectors:BEADC2012X105N -> Inductor_SMD:L_0603_1608Metric
Changed lines of the file:
@@
 F 0 "FB1" V 7553 1050 39  0000 C CNN
 F 1 "Ferrite_Bead_Small" V 7604 1050 50  0001 C CNN
-F 2 "Barrel - Audio Connectors:BEADC2012X105N" V 7680 1050 50  0001 C CNN
+F 2 "Inductor_SMD:L_0603_1608Metric" V 7680 1050 50  0001 C CNN
 F 3 "~" H 7750 1050 50  0001 C CNN
 F 4 "BLM21PG220SN1" V 7621 1050 30  0000 C CNN "MPN"
