File: src_files/mcu_ctrl.sch (KiCad schematic (older format))
At the start: 23 parts, among them J3 Conn_02x05_Odd_Even, J4 USB_B_Micro, U7 STM32F103C8Tx, U8 FXMA2104UMX, Y2 8MHz

Commit message: updated all files and production files as well
Parts:
- FB2: footprint Inductor_SMD:L_0805_2012Metric -> Inductor_SMD:L_0603_1608Metric
- U8: footprint Barrel - Audio Connectors:QFN40P180X180X55-12N -> SamacSys_Parts_2:QFN40P180X180X55-12N
Changed lines of the file:
@@
 F 0 "U8" H 2250 4700 39  0000 C CNN
 F 1 "FXMA2104UMX" H 2275 4775 39  0000 C CNN
-F 2 "Barrel - Audio Connectors:QFN40P180X180X55-12N" H 2000 5625 50  0001 L CNN
+F 2 "SamacSys_Parts_2:QFN40P180X180X55-12N" H 2000 5625 50  0001 L CNN
 F 3 "https://www.fairchildsemi.com/datasheets/FX/FXMA2104.pdf" H 2000 5725 50  0001 L CNN
 	1    2000 5225
@@
 F 0 "FB2" V 2678 2075 39  0000 C CNN
 F 1 "BLM21PG220SN1" V 2729 2075 39  0001 C CNN
-F 2 "Inductor_SMD:L_0805_2012Metric" V 2805 2075 50  0001 C CNN
+F 2 "Inductor_SMD:L_0603_1608Metric" V 2805 2075 50  0001 C CNN
 F 3 "~" H 2875 2075 50  0001 C CNN
 F 4 "FBMJ2125HS250NTV_805" V 2750 2150 30  0000 C CNN "MPN"
